File: hardware/Controle/Controle/canbus_connector.sch (KiCad schematic (older format))
At the start: 2 parts

Commit message: PCB
Parts:
- removed J?: RJ45, KicadZeniteSolarLibrary18:RJ45_YH59_01, symbol Connector:RJ45_Shielded
- gave numbers to parts that had none: 1
Changed lines of the file:
@@
 $Descr A4 11693 8268
 encoding utf-8
-Sheet 2 2
+Sheet 3 6
 Title ""
 Date ""
@@
 Comment4 ""
 $EndDescr
-Wire Wire Line
-	7500 4500 7500 3900
-Wire Wire Line
-	6550 3600 7100 3600
-Wire Wire Line
-	7100 3700 6550 3700
-Wire Wire Line
-	6550 3400 7000 3400
-Text Label 6550 3400 0    60   ~ 0
-CAN_18V
-Text Label 6550 3500 0    60   ~ 0
-CAN_GND
-Text Label 6550 3600 0    60   ~ 0
-CAN_L
-Text Label 6550 3700 0    60   ~ 0
-CAN_H
-$Comp
-L Connector:RJ45_Shielded J?
-U 1 1 5A01AFBA
-P 7500 3400
-F 0 "J?" H 7700 3950 50  0000 C CNN
-F 1 "RJ45" H 7350 3950 50  0000 C CNN
-F 2 "KicadZeniteSolarLibrary18:RJ45_YH59_01" H 7500 3400 50  0001 C CNN
-F 3 "" H 7500 3400 50  0001 C CNN
-	1    7500 3400
-	-1   0    0    -1
-$EndComp
 Text HLabel 3100 3500 0    60   BiDi ~ 0
 CAN_H
@@
 Text HLabel 3100 3700 0    60   BiDi ~ 0
 CAN_GND
-Wire Wire Line
-	7100 3000 7000 3000
-Wire Wire Line
-	6500 3000 6500 3500
-Wire Wire Line
-	6500 4500 7500 4500
-Wire Wire Line
-	7100 3100 7000 3100
-Wire Wire Line
-	7000 3100 7000 3000
-Connection ~ 7000 3000
-Wire Wire Line
-	7000 3000 6500 3000
-Wire Wire Line
-	7100 3200 7000 3200
-Wire Wire Line
-	7100 3300 7000 3300
-Wire Wire Line
-	7000 3300 7000 3400
-Connection ~ 7000 3400
-Wire Wire Line
-	7000 3400 7100 3400
-Wire Wire Line
-	6500 3500 7100 3500
-Connection ~ 6500 3500
-Wire Wire Line
-	6500 3500 6500 4500
 Wire Wire Line
 	5950 4500 5950 3900
@@
 CAN_H
 $Comp
-L Connector:RJ45_Shielded J?
+L Connector:RJ45_Shielded J301
 U 1 1 5BE6C2F7
 P 5950 3400
-F 0 "J?" H 6150 3950 50  0000 C CNN
+F 0 "J301" H 6150 3950 50  0000 C CNN
 F 1 "RJ45" H 5800 3950 50  0000 C CNN
 F 2 "KicadZeniteSolarLibrary18:RJ45_YH59_01" H 5950 3400 50  0001 C CNN
@@
 Wire Wire Line
 	4950 3500 4950 4500
-Wire Wire Line
-	5950 4500 6500 4500
-Connection ~ 5950 4500
-Connection ~ 6500 4500
 $Comp
-L power:GND #PWR?
+L power:GND #PWR0302
 U 1 1 5BE6CF28
 P 4950 4600
-F 0 "#PWR?" H 4950 4350 50  0001 C CNN
+F 0 "#PWR0302" H 4950 4350 50  0001 C CNN
 F 1 "GND" H 5000 4400 50  0000 C CNN
 F 2 "" H 4950 4600 50  0001 C CNN
@@
 	3200 3600 3100 3600
 $Comp
-L power:GND #PWR?
+L power:GND #PWR0301
 U 1 1 5BE70223
 P 3200 3800
-F 0 "#PWR?" H 3200 3550 50  0001 C CNN
+F 0 "#PWR0301" H 3200 3550 50  0001 C CNN
 F 1 "GND" H 3250 3600 50  0000 C CNN
 F 2 "" H 3200 3800 50  0001 C CNN
@@
 	5450 3200 5450 3100
 Connection ~ 5450 3100
-Wire Wire Line
-	7000 3200 7000 3100
-Connection ~ 7000 3100
 $EndSCHEMATC

Commit message: more vias!
Parts:
- J301: symbol Connector:RJ45_Shielded -> Connector:RJ45
Connections:
- net GND: no longer J301.SH
Changed lines of the file:
@@
 CAN_GND
-Wire Wire Line
-	5950 4500 5950 3900
 Wire Wire Line
 	5000 3600 5550 3600
@@
 CAN_H
 $Comp
-L Connector:RJ45_Shielded J301
+L Connector:RJ45 J301
 U 1 1 5BE6C2F7
 P 5950 3400
@@
 Wire Wire Line
 	4950 3000 4950 3500
-Wire Wire Line
-	4950 4500 5950 4500
 Wire Wire Line
 	5550 3100 5450 3100
@@
 	4950 3500 5550 3500
 Connection ~ 4950 3500
-Wire Wire Line
-	4950 3500 4950 4500
 $Comp
 L power:GND #PWR0302
@@
 	1    0    0    -1
 $EndComp
-Wire Wire Line
-	4950 4500 4950 4600
-Connection ~ 4950 4500
 Text Label 3200 3400 0    60   ~ 0
 CAN_18V
@@
 	5450 3200 5450 3100
 Connection ~ 5450 3100
+Wire Wire Line
+	4950 3500 4950 4600
 $EndSCHEMATC
