File: hardware/Caps/Caps.kicad_pcb (KiCad board)
At the start: 2 copper layers, 75 x 42 mm, 116 parts

Commit message: Gerbers re-generated with JCLJCLJLC.. string
Other:
- board text added: "JLCJLCJLCJLC"
